Commit message: fix path for mesh

File: urdf/sensors/hokuyo.urdf.xacro (robot description, xacro)
@@ -21,5 +21,5 @@
         <origin xyz="0 0 0" rpy="0 0 0"/>
         <geometry>
-          <mesh filename="package://orne_params/meshes/hokuyo.dae"/>
+          <mesh filename="package://orne_description/meshes/hokuyo.dae"/>
         </geometry>
       </visual>
