Commit message: fix/ fix typo

File: urdf/sensors/imu.urdf.xacro (robot description, xacro)
@@ -4,5 +4,5 @@
     <joint name="${name}_joint" type="fixed">
       <axis xyz="1 0 0"/>
-        <!origin xyz="0 0 0.2825"/>
+        <origin xyz="0 0 0.2825"/>
         <insert_block name="origin"/>
         <parent link="${parent}"/>
@@ -30,5 +30,5 @@
     <gazebo>
       <plugin name="ros_imu" filename="libgazebo_ros_imu.so">
-        <bodyName>imu_link</bodyName> <! bodyName always set base_link by URDF parser >
+        <bodyName>imu_link</bodyName> <!-- bodyName always set base_link by URDF parser -->
         <topicName>imu_data</topicName>
         <serviceName>imu_service</serviceName>
