Commit message: add color

File: urdf/robots/materials.xacro (robot description, xacro)
@@ -1,6 +1,13 @@
-<?xml version="1.0"?>
+<?xml version="1.0" ?>
 <robot name="xacro_properties" xmlns:xacro="http://ros.org/wiki/xacro">
+  <!-- Init colour -->
   <material name="black">
-    <color rgba="0.0 0.0 0.0 1.0"/>
+      <color rgba="0.0 0.0 0.0 1.0"/>
+  </material>
+  <material name="dark">
+    <color rgba="0.3 0.3 0.3 1.0"/>
+  </material>
+  <material name="light_black">
+    <color rgba="0.4 0.4 0.4 1.0"/>
   </material>
   <material name="blue">
@@ -11,5 +18,5 @@
   </material>
   <material name="grey">
-    <color rgba="0.2 0.2 0.2 1.0"/>
+    <color rgba="0.5 0.5 0.5 1.0"/>
   </material>
   <material name="orange">
