Commit message: Big change

File: urdf/robots/orne_alpha.gazebo.xacro (robot description, xacro)
@@ -1,45 +1,107 @@
 <?xml version="1.0"?>
-<robot>
-  <!-- ros_control plugin -->
-  <gazebo>
-    <plugin name="gazebo_ros_control" filename="libgazebo_ros_control.so">
-      <robotSimType>icart_mini_gazebo/ICartMiniHWSim</robotSimType>
-    </plugin>
+<robot name="orne_box" xmlns:xacro="http://ros.org/wiki/xacro">
+  <xacro:arg name="laser_visual" default="false"/>
+  <xacro:arg name="imu_visual"   default="false"/>
+  <gazebo reference="base_link">
+    <material>Gazebo/DarkGrey</material>
   </gazebo>
-  <!-- Left Wheel -->
-  <gazebo reference="left_wheel">
-    <mu1>1.0</mu1>
-    <mu2>1.0</mu2>
+  <gazebo reference="wheel_left_link">
+    <mu1>0.1</mu1>
+    <mu2>0.1</mu2>
+    <kp>500000.0</kp>
+    <kd>10.0</kd>
+    <minDepth>0.001</minDepth>
+    <maxVel>1.0</maxVel>
+    <fdir1>1 0 0</fdir1>
+    <material>Gazebo/FlatBlack</material>
+  </gazebo>
+  <gazebo reference="wheel_right_link">
+    <mu1>0.1</mu1>
+    <mu2>0.1</mu2>
+    <kp>500000.0</kp>
+    <kd>10.0</kd>
+    <minDepth>0.001</minDepth>
+    <maxVel>1.0</maxVel>
+    <fdir1>1 0 0</fdir1>
+    <material>Gazebo/FlatBlack</material>
+  </gazebo>
+  <gazebo reference="caster_front_link">
+    <mu1>0.1</mu1>
+    <mu2>0.1</mu2>
     <kp>1000000.0</kp>
     <kd>100.0</kd>
     <minDepth>0.001</minDepth>
     <maxVel>1.0</maxVel>
-    <material>Gazebo/Orange</material>
+    <material>Gazebo/FlatBlack</material>
   </gazebo>
-  <!-- Base Link -->
-  <gazebo reference="base_link">
-    <material>Gazebo/White</material>
+  <gazebo reference="imu_link">
+    <sensor type="imu" name="imu">
+      <always_on>true</always_on>
+      <visualize>$(arg imu_visual)</visualize>
+    </sensor>
+    <material>Gazebo/FlatBlack</material>
   </gazebo>
-  <!-- Right Wheel -->
-  <gazebo reference="right_wheel">
-    <mu1>1.0</mu1>
-    <mu2>1.0</mu2>
-    <kp>1000000.0</kp>
-    <kd>100.0</kd>
-    <minDepth>0.001</minDepth>
-    <maxVel>1.0</maxVel>
-    <material>Gazebo/Orange</material>
+  <gazebo>
+    <plugin name="orne_box_controller" filename="libgazebo_ros_diff_drive.so">
+      <commandTopic>icart_mini/cmd_vel</commandTopic>
+      <odometryTopic>icart_mini/odom</odometryTopic>
+      <odometryFrame>odom</odometryFrame>
+      <odometrySource>world</odometrySource>
+      <publishOdomTF>true</publishOdomTF>
+      <robotBaseFrame>base_footprint</robotBaseFrame>
+      <publishWheelTF>true</publishWheelTF>
+      <publishTf>true</publishTf>
+      <publishWheelJointState>true</publishWheelJointState>
+      <legacyMode>false</legacyMode>
+      <updateRate>30</updateRate>
+      <leftJoint>wheel_left_joint</leftJoint>
+      <rightJoint>wheel_right_joint</rightJoint>
+      <wheelSeparation>0.4615</wheelSeparation>
+      <wheelDiameter>0.304</wheelDiameter>
+      <wheelAcceleration>1</wheelAcceleration>
+      <wheelTorque>10</wheelTorque>
+      <rosDebugLevel>na</rosDebugLevel>
+    </plugin>
   </gazebo>
-  <!-- hokuyo -->
-  <gazebo reference="hokuyo_link">
-    <sensor type="ray" name="head_hokuyo_sensor">
+  <gazebo>
+    <plugin name="imu_plugin" filename="libgazebo_ros_imu.so">
+      <alwaysOn>true</alwaysOn>
+      <bodyName>imu_link</bodyName>
+      <frameName>imu_link</frameName>
+      <topicName>imu</topicName>
+      <serviceName>imu_service</serviceName>
+      <gaussianNoise>0.0</gaussianNoise>
+      <updateRate>200</updateRate>
+      <imu>
+        <noise>
+          <type>gaussian</type>
+          <rate>
+            <mean>0.0</mean>
+            <stddev>2e-4</stddev>
+            <bias_mean>0.0000075</bias_mean>
+            <bias_stddev>0.0000008</bias_stddev>
+          </rate>
+          <accel>
+            <mean>0.0</mean>
+            <stddev>1.7e-2</stddev>
+            <bias_mean>0.1</bias_mean>
+            <bias_stddev>0.001</bias_stddev>
+          </accel>
+        </noise>
+      </imu>
+    </plugin>
+  </gazebo>
+  <!--UTM-30-LX specifications-->
+  <gazebo reference="base_scan">
+    <material>Gazebo/FlatBlack</material>
+    <sensor type="ray" name="lds_lfcd_sensor">
       <pose>0 0 0 0 0 0</pose>
-      <visualize>false</visualize>
-      <update_rate>40</update_rate>
+      <visualize>$(arg laser_visual)</visualize>
+      <update_rate>5</update_rate>
       <ray>
         <scan>
           <horizontal>
             <samples>720</samples>
-            <resolution>1</resolution>
+            <resolution>0.25</resolution>
             <min_angle>-1.570796</min_angle>
             <max_angle>1.570796</max_angle>
@@ -47,21 +109,17 @@
         </scan>
         <range>
-          <min>0.10</min>
+          <min>0.1</min>
           <max>30.0</max>
-          <resolution>0.01</resolution>
+          <resolution>0.05</resolution>
         </range>
         <noise>
           <type>gaussian</type>
-          <!-- Noise parameters based on published spec for Hokuyo laser
-               achieving "+-30mm" accuracy at range < 10m.  A mean of 0.0m and
-               stddev of 0.01m will put 99.7% of samples within 0.03m of the true
-               reading. -->
           <mean>0.0</mean>
           <stddev>0.01</stddev>
         </noise>
       </ray>
-      <plugin name="gazebo_ros_head_hokuyo_controller" filename="libgazebo_ros_laser.so">
-        <topicName>/scan</topicName>
-        <frameName>hokuyo_link</frameName>
+      <plugin name="gazebo_ros_lds_lfcd_controller" filename="libgazebo_ros_laser.so">
+        <topicName>scan</topicName>
+        <frameName>base_scan</frameName>
       </plugin>
     </sensor>

File: urdf/robots/orne_alpha.urdf.xacro (robot description, xacro)
@@ -1,170 +1,140 @@
-<?xml version="1.0"?>
-<robot name="orne_alpha" xmlns:xacro="http://ros.org/wiki/xacro">
-  <!-- Constants for robot dimensions -->
-  <xacro:property name="PI" value="3.1415926535897931"/>
-  <!-- Import Rviz colors -->
-  <xacro:include filename="$(find orne_description)/urdf/robots/materials.xacro" />
+<?xml version="1.0" ?>
+<robot name="orne" xmlns:xacro="http://ros.org/wiki/xacro">
+  <xacro:include filename="$(find orne_description)/urdf/robots/materials.xacro"/>
   <xacro:include filename="$(find orne_description)/urdf/robots/orne_alpha.gazebo.xacro"/>
-  <xacro:include filename="$(find orne_description)/urdf/sensors/imu.urdf.xacro"/>
-  <xacro:include filename="$(find orne_description)/urdf/sensors/hokuyo.urdf.xacro"/>
-  <!-- Setting for imu -->
-  <xacro:sensor_imu name="imu" parent="base_link" size="0.05 0.05 0.05">
-    <origin xyz="-0.145 0.0 0.21" rpy="0 3.14 0"/>
-  </xacro:sensor_imu>
-  <!-- Setting for 2D URG -->
-  <xacro:sensor_hokuyo name="hokuyo" parent="base_link">
-    <origin xyz="0.212 0 0.2485" rpy="0 0 0"/>
-  </xacro:sensor_hokuyo>
-  <!-- Setting for Velodyne -->
-  <xacro:include filename="$(find orne_description)/urdf/sensors/vlp16.urdf.xacro"/>
-  <xacro:VLP-16 name="velodyne" parent="base_link">
-    <origin xyz="0.098 0.0 0.422" rpy="0 0 -0.12"/>
-  </xacro:VLP-16>
-<!-- Setting for ORNE alpha -->
-  <!-- Base Link -->
+  <link name="base_footprint"/>
+  <joint name="base_joint" type="fixed">
+    <parent link="base_footprint"/>
+    <child link="base_link"/>
+    <origin xyz="0.0 0.0 0.152" rpy="0 0 0"/>
+  </joint>
   <link name="base_link">
-    <collision>
-      <origin xyz="0 0 0.1" rpy="0 0 0"/>
+    <visual>
+      <origin xyz="0.0 0 0" rpy="0 0 0"/>
       <geometry>
-           <box size=".40 .45 .134"/>
+        <mesh filename="package://orne_description/meshes/bases/orne_alpha_base.stl" scale="1 1 1"/>
       </geometry>
-    </collision>
-    <visual>
-      <origin xyz="0.1 0 0.1" rpy="0 0 0"/>
-      <geometry>
-           <box size=".40 .45 .134"/>
-      </geometry>
-      <material name="orange"/>
+      <material name="light_black"/>
     </visual>
     <collision>
-      <origin xyz="0.005 0 0.305" rpy="0 0 0"/>
+      <origin xyz="0.158 0 0" rpy="0 0 0"/>
       <geometry>
-           <box size=".376 .45 .134"/>
-      </geometry>
-    </collision>
-    <visual>
-      <origin xyz="0.005 0 0.305" rpy="0 0 0"/>
-      <geometry>
-           <box size=".376 .45 .134"/>
-      </geometry>
-      <material name="orange"/>
-    </visual>
-    <collision name="collision">
-      <origin xyz="0.301 -0.141 0.075" rpy="0 1.5707 1.5707"/>
-      <geometry>
-        <cylinder  length="0.03" radius="0.075"/>
-      </geometry>
-    </collision>
-    <visual name="visual">
-      <origin xyz="0.301 -0.141 0.075" rpy="0 1.5707 1.5707"/>
-      <geometry>
-        <cylinder  length="0.03" radius="0.075"/>
-      </geometry>
-    </visual>
-    <collision name="collision">
-      <origin xyz="0.301 0.141 0.075" rpy="0 1.5707 1.5707"/>
-      <geometry>
-        <cylinder  length="0.03" radius="0.075"/>
-      </geometry>
-    </collision>
-    <visual name="visual">
-      <origin xyz="0.301 0.141 0.075" rpy="0 1.5707 1.5707"/>
-      <geometry>
-        <cylinder  length="0.03" radius="0.075"/>
-      </geometry>
-    </visual>
-    <inertial>
-       <mass value="15" />
-       <origin xyz="0 0 0" rpy="0 0 0"/>
-       <inertia ixx="1" ixy="0" ixz="0" iyy="1" iyz="0" izz="1" />
-    </inertial>
-  </link>
-  <link name="visual_left_wheel">
-    <visual name="visual">
-      <origin xyz="0 0.0 0" rpy="0 1.5707 1.5707"/>
-      <geometry>
-        <cylinder  length="0.03" radius="0.151"/>
-      </geometry>
-    </visual>
-  </link>
-  <joint type="fixed" name="visual_left_wheel_hinge">
-    <origin xyz="-0.045 0.233 0.1518" rpy="0 0 0"/>
-    <child link="visual_left_wheel">visual_left_wheel</child>
-    <parent link="base_link">base_link</parent>
-    <axis xyz="0 1 0"/>
-  </joint>
-  <link name="left_wheel">
-    <collision name="collision">
-      <origin xyz="0 0.0 0" rpy="0 1.5707 1.5707"/>
-      <geometry>
-         <cylinder  length="0.03" radius="0.151"/>
+        <box size="0.70 0.40 0.02"/>
       </geometry>
     </collision>
     <inertial>
-      <mass value="1" />
-      <origin xyz="0 0.0 0"/>
-      <inertia ixx="0.1" ixy="0" ixz="0" iyy="0.1" iyz="0" izz="0.1" />
+      <origin xyz="0 0 0" rpy="0 0 0"/>
+      <mass value="15.0"/>
+      <inertia ixx="0.001" ixy="0.0" ixz="0.0"
+               iyy="0.001" iyz="0.0"
+               izz="0.001" />
     </inertial>
   </link>
-  <joint type="revolute" name="left_wheel_hinge">
-    <origin xyz="-0.045 0.223 0.1518" rpy="0 0 0"/>
-    <child link="left_wheel">left_wheel</child>
-    <parent link="base_link">base_link</parent>
-    <axis xyz="0 1 0"/>
-    <limit effort="100" velocity="100.0"  lower="-5000" upper="5000" />
+  <joint name="wheel_left_joint" type="continuous">
+    <parent link="base_link"/>
+    <child link="wheel_left_link"/>
+    <origin xyz="0.0 0.23075 0.0" rpy="-1.57 0 0"/>
+    <axis xyz="0 0 1"/>
   </joint>
-  <link name="visual_right_wheel">
-    <visual name="visual">
-      <origin xyz="0 0.0 0" rpy="0 1.5707 1.5707"/>
+  <link name="wheel_left_link">
+    <visual>
+      <origin xyz="0 0 0" rpy="0 3.14 0"/>
       <geometry>
-        <cylinder  length="0.03" radius="0.151"/>
+        <mesh filename="package://orne_description/meshes/wheels/tire.stl" scale="1 1 1"/>
       </geometry>
+      <material name="dark"/>
     </visual>
-  </link>
-  <joint type="fixed" name="visual_right_wheel_hinge">
-    <origin xyz="-0.045 -0.223 0.1518" rpy="0 0 0"/>
-    <child link="visual_right_wheel">visual_right_wheel</child>
-    <parent link="base_link">base_link</parent>
-    <axis xyz="0 1 0"/>
-  </joint>
-  <link name="right_wheel">
-    <collision name="collision">
-      <origin xyz="0 0.0 0" rpy="0 1.5707 1.5707"/>
+    <collision>
+      <origin xyz="0 0 0" rpy="0 0 0"/>
       <geometry>
-         <cylinder  length="0.03" radius="0.151"/>
+        <cylinder length="0.0225" radius="0.152"/>
       </geometry>
     </collision>
     <inertial>
-      <mass value="1" />
-      <origin xyz="0 0.0 0"/>
-      <inertia ixx="0.1" ixy="0" ixz="0" iyy="0.1" iyz="0" izz="0.1" />
+      <origin xyz="0 0 0" />
+      <mass value="0.2" />
+        <inertia ixx="0.001" ixy="0.0" ixz="0.0"
+                 iyy="0.001" iyz="0.0"
+                 izz="0.001" />
     </inertial>
   </link>
-  <joint type="revolute" name="right_wheel_hinge">
-    <origin xyz="-0.045 -0.223 0.1518" rpy="0 0 0"/>
-    <child link="right_wheel">right_wheel</child>
-    <parent link="base_link">base_link</parent>
-    <axis xyz="0 1 0"/>
-    <limit effort="100" velocity="100.0"  lower="-5000" upper="5000" />
+  <joint name="wheel_right_joint" type="continuous">
+    <parent link="base_link"/>
+    <child link="wheel_right_link"/>
+    <origin xyz="0.0 -0.23075 0.0" rpy="-1.57 0 0"/>
+    <axis xyz="0 0 1"/>
   </joint>
-  <transmission name="tran1">
-    <type>transmission_interface/SimpleTransmission</type>
-    <joint name="left_wheel_hinge">
-      <hardwareInterface>VelocityJointInterface</hardwareInterface>
-    </joint>
-  <actuator name="left_motor">
-      <hardwareInterface>VelocityJointInterface</hardwareInterface>
-      <mechanicalReduction>1</mechanicalReduction>
-    </actuator>
-  </transmission>
-  <transmission name="tran2">
-    <type>transmission_interface/SimpleTransmission</type>
-    <joint name="right_wheel_hinge">
-      <hardwareInterface>VelocityJointInterface</hardwareInterface>
-    </joint>
-  <actuator name="right_motor">
-      <hardwareInterface>VelocityJointInterface</hardwareInterface>
-      <mechanicalReduction>1</mechanicalReduction>
-    </actuator>
-  </transmission>
+  <link name="wheel_right_link">
+    <visual>
+      <origin xyz="0 0 0" rpy="0 0 0"/>
+      <geometry>
+        <mesh filename="package://orne_description/meshes/wheels/tire.stl" scale="1 1 1"/>
+      </geometry>
+      <material name="dark"/>
+    </visual>
+    <collision>
+      <origin xyz="0 0 0" rpy="0 0 0"/>
+      <geometry>
+        <cylinder length="0.0225" radius="0.152"/>
+      </geometry>
+    </collision>
+      <inertial>
+        <origin xyz="0 0 0" />
+        <mass value="0.2" />
+        <inertia ixx="0.001" ixy="0.0" ixz="0.0"
+                 iyy="0.001" iyz="0.0"
+                 izz="0.001" />
+      </inertial>
+  </link>
+  <joint name="caster_front_joint" type="fixed">
+    <parent link="base_link"/>
+    <child link="caster_front_link"/>
+    <origin xyz="0.374295 0 0.015" rpy="-3.14 0 0"/>
+  </joint>
+  <link name="caster_front_link">
+    <collision>
+      <origin xyz="0 0.0 0.0835" rpy="0 0 0"/>
+      <geometry>
+        <box size="0.10 0.4 0.167"/>
+      </geometry>
+    </collision>
+    <inertial>
+      <origin xyz="0 0 0" />
+      <mass value="1.0" />
+      <inertia ixx="0.001" ixy="0.0" ixz="0.0"
+               iyy="0.001" iyz="0.0"
+               izz="0.001" />
+    </inertial>
+  </link>
+  <joint name="imu_joint" type="fixed">
+    <parent link="base_link"/>
+    <child link="imu_link"/>
+    <origin xyz="0 0 0" rpy="0 0 0"/>
+  </joint>
+  <link name="imu_link"/>
+  <joint name="scan_joint" type="fixed">
+    <parent link="base_link"/>
+    <child link="base_scan"/>
+    <origin xyz="0.374295 0 0.1225" rpy="0 0 0"/>
+  </joint>
+  <link name="base_scan">
+     <visual>
+      <origin xyz="-0.0125 0 -0.035" rpy="1.57 0 1.57"/>
+      <geometry>
+        <mesh filename="package://orne_description/meshes/sensors/UTM-30LX_LN.stl" scale="0.01 0.01 0.01"/>
+      </geometry>
+      <material name="dark"/>
+    </visual>
+    <inertial>
+      <mass value="0.08" />
+      <origin xyz="0 0 0" />
+      <inertia ixx="0.001" ixy="0.0" ixz="0.0"
+               iyy="0.001" iyz="0.0"
+               izz="0.001" />
+    </inertial>
+  </link>
+  <xacro:include filename="$(find velodyne_description)/urdf/VLP-16.urdf.xacro"/>
+  <xacro:VLP-16 parent="base_scan" name="velodyne" topic="/velodyne_points" hz="10" samples="440">
+  <origin xyz="-0.10 0 0.15" rpy="0 0 0" />
+  </xacro:VLP-16>
 </robot>
